Commit message: fix: issues with contact forces were caused by the urdf format

File: legged_gym/resources/robots/silver_badger/urdf/intention.urdf (robot description, URDF)
Before this commit: robot intention, 19 links, 18 joints
Joints:
- joint fl_jFoot: axis 0.0 0 0 -> (none)
- joint fr_jFoot: axis 0.0 0 0 -> (none)
- joint rl_jFoot: axis 0.0 0 0 -> (none)
- joint root: axis 0 0 0 -> (none); type floating -> fixed
- joint rr_jFoot: axis 0.0 0 0 -> (none)

Commit message: Modify config. Modify urdf file to lock the spine

File: legged_gym/resources/robots/silver_badger/urdf/intention.urdf (robot description, URDF)
Before this commit: robot intention, 19 links, 18 joints
Joints:
- joint fl_j0: type continuous -> revolute
- joint fl_j1: type continuous -> revolute
- joint fl_j2: type continuous -> revolute
- joint fr_j0: type continuous -> revolute
- joint fr_j1: type continuous -> revolute
- joint fr_j2: type continuous -> revolute
- joint rl_j0: type continuous -> revolute
- joint rl_j1: type continuous -> revolute
- joint rl_j2: type continuous -> revolute
- joint rr_j0: type continuous -> revolute
- joint rr_j1: type continuous -> revolute
- joint rr_j2: type continuous -> revolute
- joint sp_j0: type continuous -> fixed

Commit message: Change spine joint to revolute. Modify armature and thickness.

File: legged_gym/resources/robots/silver_badger/urdf/intention.urdf (robot description, URDF)
Before this commit: robot intention, 19 links, 18 joints
Joints:
- joint sp_j0: limit lower=-0.785 upper=0.785 effort=48.0 velocity=3.15 -> lower=-0.001 upper=0.001 effort=48.0 velocity=3.15; type fixed -> revolute
